File: PCB/PCBV2/PCBV2.kicad_pcb (KiCad board)
At the start: 2 copper layers, 368.3 x 121.9 mm, 225 parts, among them SW1 SW_PUSH, SW2 SW_PUSH, U1 STM32F072CBUx, U2 MCP1700-3302E_SOT23, U3 USBLC6-2SC6

Commit message: Minor Updates
Parts:
- K_90: footprint MX_Only:MXOnly-6.25U-NoLED -> MX_Only:MXOnly-6.25U-ReversedStabilizers-NoLED
- moved C1 2.40 mm to (271.4, 190.3)
- moved C5 2.40 mm to (270.2, 190.3)
Routing:
- net row0: track 667.1 -> 673.0 mm
- net +3V3: track 343.7 -> 348.3 mm
- net GND: track 404.0 -> 405.8 mm
- net BOOT0: track 237.4 -> 238.2 mm
- net Net-(D_93-Pad2): track 25.9 -> 26.6 mm
- net row5: track 525.4 -> 526.1 mm
Other:
- rule trace_min: 0.2 -> 0

Commit message: BIG CHANGES
Parts:
- added D_101: D, Diode_SMD:D_SOD-123, B.Cu at (109.5, 173.8)
- added D_90: D, Diode_SMD:D_SOD-123, B.Cu at (373.9, 142.1)
- added K_101: KEYSW, MX_Only:MXOnly-1.25U-NoLED, F.Cu at (101.6, 149.2)
- added K_ISO1u1R1: KEYSW, MX_Only:MXOnly-1U-NoLED, F.Cu at (342.1, 149.2)
- added K_ISO1uL1: KEYSW, MX_Only:MXOnly-1U-NoLED, F.Cu at (123.0, 168.3)
- added K_ISOEnter1: KEYSW, MX_Only:MXOnly-ISO-ReversedStabilizers, F.Cu at (363.5, 139.7)
- added K_ISOShift1: KEYSW, MX_Only:MXOnly-1.25U-NoLED, F.Cu at (101.6, 168.3)
- K_90: footprint MX_Only:MXOnly-6.25U-ReversedStabilizers-NoLED -> MX_Only:MXOnly-6.25U-NoLED
- moved D_66 2.17 mm to (373.9, 147.6), turned to 180 degrees
- renumbered K_49 to K_49ANSISlash1, K_66 to K_ANSIEnter1, K_70 to K_ANSIShift1
Routing:
- net row4: track 536.6 -> 558.3 mm
- net row3: track 566.0 -> 584.4 mm
- net Net-(D_66-Pad2): track 19.5 -> 32.8 mm
- net Net-(D_101-Pad2): track 0.00 -> 12.2 mm
- net col13: track 186.4 -> 198.3 mm
- net Net-(D_90-Pad2): track 0.00 -> 10.00 mm
- net Net-(D_70-Pad2): track 19.5 -> 27.1 mm
- net col0: track 292.5 -> 299.9 mm
- net col1: track 270.0 -> 276.6 mm
- net Net-(D_54-Pad2): track 15.2 -> 19.9 mm
- net col14: track 191.6 -> 195.1 mm
- net BOOT0: track 238.2 -> 241.3 mm
- net NRST: track 219.7 -> 221.7 mm
