File: PCB/PCBV2/PCBV2.sch (KiCad schematic (older format))
At the start: 225 parts, among them SW1 SW_PUSH, SW2 SW_PUSH, U1 STM32F072CBUx, U2 MCP1700-3302E_SOT23, U3 USBLC6-2SC6

Commit message: BIG CHANGES
Parts:
- added D_101, D_90: D, Diode_SMD:D_SOD-123, symbol Device:D_Small
- added K_101, K_ISOShift1: KEYSW, MX_Only:MXOnly-1.25U-NoLED, symbol MX_Alps_Hybrid:MX-NoLED
- added K_ISO1u1R1, K_ISO1uL1: KEYSW, MX_Only:MXOnly-1U-NoLED, symbol MX_Alps_Hybrid:MX-NoLED
- added K_ISOEnter1: KEYSW, MX_Only:MXOnly-ISO-ReversedStabilizers, symbol MX_Alps_Hybrid:MX-NoLED
- K_90: footprint MX_Only:MXOnly-6.25U-ReversedStabilizers-NoLED -> MX_Only:MXOnly-6.25U-NoLED
- renumbered K_49 to K_49ANSISlash1, K_66 to K_ANSIEnter1, K_70 to K_ANSIShift1
Connections:
- net col0: now also K_101.1 (COL), K_ISOShift1.1 (COL)
- net col1: now also K_ISO1uL1.1 (COL)
- net col13: now also K_ISO1u1R1.1 (COL)
- net col14: now also K_ISOEnter1.1 (COL)
- net row3: now also D_90.1 (K)
- net row4: now also D_101.1 (K)
- net at D_54.2 (A), K_54.2 (ROW): now also K_101.2 (ROW)
- net at D_66.2 (A), K_ANSIEnter1.2 (ROW): now also K_ISO1u1R1.2 (ROW)
- net at D_70.2 (A), K_ANSIShift1.2 (ROW): now also K_ISO1uL1.2 (ROW)
- new net: D_90.2 (A), K_ISOEnter1.2 (ROW)
- new net: D_101.2 (A), K_ISOShift1.2 (ROW)
Changed lines of the file:
@@
 Connection ~ 16050 11200
 $Comp
-L MX_Alps_Hybrid:MX-NoLED K_49
+L MX_Alps_Hybrid:MX-NoLED K_49ANSISlash1
 U 1 1 00000491
 P 17100 10800
-F 0 "K_49" H 17100 11033 60  0000 C CNN
+F 0 "K_49ANSISlash1" H 17100 11033 60  0000 C CNN
 F 1 "KEYSW" H 17100 10700 60  0001 C CNN
 F 2 "MX_Only:MXOnly-1.5U-NoLED" H 17100 10800 60  0001 C CNN
@@
 $EndComp
 Wire Wire Line
-	3250 11750 3500 11750
+	3250 11750 3350 11750
 Wire Wire Line
 	3050 11950 3050 12000
@@
 Connection ~ 15050 12200
 $Comp
-L MX_Alps_Hybrid:MX-NoLED K_66
-U 1 1 00000661
-P 16100 11800
-F 0 "K_66" H 16100 12033 60  0000 C CNN
-F 1 "KEYSW" H 16100 11700 60  0001 C CNN
-F 2 "MX_Only:MXOnly-2.25U-NoLED" H 16100 11800 60  0001 C CNN
-F 3 "" H 16100 11800 60  0000 C CNN
-	1    16100 11800
-	1    0    0    -1
-$EndComp
-$Comp
 L Device:D_Small D_66
 U 1 1 00000660
@@
 row4
 $Comp
-L MX_Alps_Hybrid:MX-NoLED K_70
+L MX_Alps_Hybrid:MX-NoLED K_ANSIShift1
 U 1 1 00000701
 P 4100 12800
-F 0 "K_70" H 4100 13033 60  0000 C CNN
+F 0 "K_ANSIShift1" H 4100 13033 60  0000 C CNN
 F 1 "KEYSW" H 4100 12700 60  0001 C CNN
 F 2 "MX_Only:MXOnly-2.25U-NoLED" H 4100 12800 60  0001 C CNN
@@
 Connection ~ 15050 13200
 $Comp
-L MX_Alps_Hybrid:MX-NoLED K_82
-U 1 1 00000821
-P 17100 12800
-F 0 "K_82" H 17100 13033 60  0000 C CNN
-F 1 "KEYSW" H 17100 12700 60  0001 C CNN
-F 2 "MX_Only:MXOnly-1U-NoLED" H 17100 12800 60  0001 C CNN
-F 3 "" H 17100 12800 60  0000 C CNN
-	1    17100 12800
-	1    0    0    -1
-$EndComp
-$Comp
-L Device:D_Small D_82
-U 1 1 00000820
-P 17050 13100
-F 0 "D_82" V 17120 13000 50  0000 R CNN
-F 1 "D" V 17030 13000 50  0000 R CNN
-F 2 "Diode_SMD:D_SOD-123" H 16750 13050 50  0001 C CNN
-F 3 "~" H 16750 13050 50  0001 C CNN
-	1    17050 13100
-	0    -1   -1   0
-$EndComp
-Wire Wire Line
-	17250 12750 17500 12750
-Wire Wire Line
-	17050 12950 17050 13000
-Connection ~ 17500 12750
-Connection ~ 17050 13200
-$Comp
 L MX_Alps_Hybrid:MX-NoLED K_83
 U 1 1 00000831
@@
 F 0 "K_90" H 8700 14033 60  0000 C CNN
 F 1 "KEYSW" H 8700 13700 60  0001 C CNN
-F 2 "MX_Only:MXOnly-6.25U-ReversedStabilizers-NoLED" H 8700 13800 60  0001 C CNN
+F 2 "MX_Only:MXOnly-6.25U-NoLED" H 8700 13800 60  0001 C CNN
 F 3 "" H 8700 13800 60  0000 C CNN
 	1    8700 13800
@@
 	21050 13950 21050 14000
 Wire Wire Line
-	3500 13750 3500 11750
+	3500 13750 3500 12700
 Wire Wire Line
 	4500 13750 4500 12750
@@
 	15500 13750 15500 12750
 Wire Wire Line
-	16500 11750 16500 10750
-Wire Wire Line
-	17500 13750 17500 12750
-Wire Wire Line
 	18500 13750 18500 12750
 Wire Wire Line
@@
 	15500 11750 15500 10750
 Wire Wire Line
-	15050 12200 16050 12200
-Wire Wire Line
-	16050 12200 18050 12200
-Wire Wire Line
 	18500 11750 18500 10750
 Wire Wire Line
@@
 	21500 11750 21500 9750
 Wire Wire Line
-	4500 12750 4500 9750
-Wire Wire Line
 	4050 13200 5050 13200
 Wire Wire Line
@@
 	15500 12750 15500 11750
 Wire Wire Line
-	15050 13200 17050 13200
-Wire Wire Line
-	17500 12750 17500 10750
-Wire Wire Line
-	17050 13200 18050 13200
-Wire Wire Line
 	18500 12750 18500 11750
 Wire Wire Line
@@
 	3050 12200 5050 12200
 Wire Wire Line
-	2600 13200 4050 13200
+	2600 13200 3100 13200
 Wire Wire Line
 	3050 14200 4050 14200
@@
 Wire Wire Line
 	14950 2300 15200 2300
+$Comp
+L MX_Alps_Hybrid:MX-NoLED K_101
+U 1 1 5F9FF284
+P 2500 11800
+F 0 "K_101" H 2500 12033 60  0000 C CNN
+F 1 "KEYSW" H 2500 11700 60  0001 C CNN
+F 2 "MX_Only:MXOnly-1.25U-NoLED" H 2500 11800 60  0001 C CNN
+F 3 "" H 2500 11800 60  0000 C CNN
+	1    2500 11800
+	1    0    0    -1
+$EndComp
+Wire Wire Line
+	2650 11750 2900 11750
+Wire Wire Line
+	2900 11750 2900 11450
+Wire Wire Line
+	2900 11450 3350 11450
+Wire Wire Line
+	3350 11450 3350 11750
+Connection ~ 3350 11750
+Wire Wire Line
+	3350 11750 3500 11750
+Wire Wire Line
+	2450 11950 2450 12000
+Wire Wire Line
+	2450 12000 3050 12000
+Connection ~ 3050 12000
+Wire Wire Line
+	15050 12200 16050 12200
+Wire Wire Line
+	17500 13750 17500 12750
+Connection ~ 17500 12750
+Wire Wire Line
+	17250 12750 17500 12750
+Wire Wire Line
+	17050 13200 18050 13200
+Connection ~ 17050 13200
+$Comp
+L Device:D_Small D_82
+U 1 1 00000820
+P 17050 13100
+F 0 "D_82" V 17120 13000 50  0000 R CNN
+F 1 "D" V 17030 13000 50  0000 R CNN
+F 2 "Diode_SMD:D_SOD-123" H 16750 13050 50  0001 C CNN
+F 3 "~" H 16750 13050 50  0001 C CNN
+	1    17050 13100
+	0    -1   -1   0
+$EndComp
+Wire Wire Line
+	17050 12950 17050 13000
+$Comp
+L MX_Alps_Hybrid:MX-NoLED K_82
+U 1 1 00000821
+P 17100 12800
+F 0 "K_82" H 17100 13033 60  0000 C CNN
+F 1 "KEYSW" H 17100 12700 60  0001 C CNN
+F 2 "MX_Only:MXOnly-1U-NoLED" H 17100 12800 60  0001 C CNN
+F 3 "" H 17100 12800 60  0000 C CNN
+	1    17100 12800
+	1    0    0    -1
+$EndComp
+Wire Wire Line
+	15050 13200 17050 13200
+Wire Wire Line
+	16050 12200 17100 12200
+Wire Wire Line
+	17500 12750 17500 11700
+$Comp
+L MX_Alps_Hybrid:MX-NoLED K_ANSIEnter1
+U 1 1 00000661
+P 16100 11800
+F 0 "K_ANSIEnter1" H 16100 12033 60  0000 C CNN
+F 1 "KEYSW" H 16100 11700 60  0001 C CNN
+F 2 "MX_Only:MXOnly-2.25U-NoLED" H 16100 11800 60  0001 C CNN
+F 3 "" H 16100 11800 60  0000 C CNN
+	1    16100 11800
+	1    0    0    -1
+$EndComp
+Wire Wire Line
+	15700 12000 16050 12000
+Connection ~ 16050 12000
+$Comp
+L Device:D_Small D_90
+U 1 1 5FDDB57C
+P 17100 12100
+F 0 "D_90" V 17170 12000 50  0000 R CNN
+F 1 "D" V 17080 12000 50  0000 R CNN
+F 2 "Diode_SMD:D_SOD-123" H 16800 12050 50  0001 C CNN
+F 3 "~" H 16800 12050 50  0001 C CNN
+	1    17100 12100
+	0    -1   -1   0
+$EndComp
+Connection ~ 17100 12200
+Wire Wire Line
+	17100 12200 18050 12200
+Wire Wire Line
+	17100 11900 17100 12000
+Wire Wire Line
+	17300 11700 17500 11700
+Connection ~ 17500 11700
+Wire Wire Line
+	17500 11700 17500 10750
+$Comp
+L MX_Alps_Hybrid:MX-NoLED K_ISOEnter1
+U 1 1 5FDDAEEA
+P 17150 11750
+F 0 "K_ISOEnter1" H 17150 11983 60  0000 C CNN
+F 1 "KEYSW" H 17150 11650 60  0001 C CNN
+F 2 "MX_Only:MXOnly-ISO-ReversedStabilizers" H 17150 11750 60  0001 C CNN
+F 3 "" H 17150 11750 60  0000 C CNN
+	1    17150 11750
+	1    0    0    -1
+$EndComp
+$Comp
+L MX_Alps_Hybrid:MX-NoLED K_ISOShift1
+U 1 1 5FEE39B3
+P 3150 12750
+F 0 "K_ISOShift1" H 3150 12983 60  0000 C CNN
+F 1 "KEYSW" H 3150 12650 60  0001 C CNN
+F 2 "MX_Only:MXOnly-1.25U-NoLED" H 3150 12750 60  0001 C CNN
+F 3 "" H 3150 12750 60  0000 C CNN
+	1    3150 12750
+	1    0    0    -1
+$EndComp
+Wire Wire Line
+	4500 9750 4500 12600
+Wire Wire Line
+	3300 12700 3500 12700
+Connection ~ 3500 12700
+Wire Wire Line
+	3500 12700 3500 11750
+$Comp
+L Device:D_Small D_101
+U 1 1 5FFBA630
+P 3100 13100
+F 0 "D_101" V 3170 13000 50  0000 R CNN
+F 1 "D" V 3080 13000 50  0000 R CNN
+F 2 "Diode_SMD:D_SOD-123" H 2800 13050 50  0001 C CNN
+F 3 "~" H 2800 13050 50  0001 C CNN
+	1    3100 13100
+	0    -1   -1   0
+$EndComp
+Connection ~ 3100 13200
+Wire Wire Line
+	3100 13200 4050 13200
+Wire Wire Line
+	3100 12900 3100 13000
+$Comp
+L MX_Alps_Hybrid:MX-NoLED K_ISO1uL1
+U 1 1 6000220A
+P 3750 12650
+F 0 "K_ISO1uL1" H 3750 12883 60  0000 C CNN
+F 1 "KEYSW" H 3750 12550 60  0001 C CNN
+F 2 "MX_Only:MXOnly-1U-NoLED" H 3750 12650 60  0001 C CNN
+F 3 "" H 3750 12650 60  0000 C CNN
+	1    3750 12650
+	1    0    0    -1
+$EndComp
+Wire Wire Line
+	3900 12600 4500 12600
+Connection ~ 4500 12600
+Wire Wire Line
+	4500 12600 4500 12750
+Wire Wire Line
+	3700 13000 4050 13000
+Connection ~ 4050 13000
+Wire Wire Line
+	16500 10750 16500 11600
+$Comp
+L MX_Alps_Hybrid:MX-NoLED K_ISO1u1R1
+U 1 1 5FD50D9F
+P 15750 11650
+F 0 "K_ISO1u1R1" H 15750 11883 60  0000 C CNN
+F 1 "KEYSW" H 15750 11550 60  0001 C CNN
+F 2 "MX_Only:MXOnly-1U-NoLED" H 15750 11650 60  0001 C CNN
+F 3 "" H 15750 11650 60  0000 C CNN
+	1    15750 11650
+	1    0    0    -1
+$EndComp
+Wire Wire Line
+	15900 11600 16500 11600
+Connection ~ 16500 11600
+Wire Wire Line
+	16500 11600 16500 11750
+Wire Wire Line
+	15700 11800 15700 12000
+Wire Wire Line
+	3700 12800 3700 13000
 $EndSCHEMATC
