File: PCB/PCBV3/PCBV3.kicad_pcb (KiCad board)
At the start: 2 copper layers, 368.3 x 121.9 mm, 232 parts, among them SW1 SW_PUSH, SW2 SW_PUSH, U1 STM32F072CBUx, U2 MCP1700-3302E_SOT23, U3 USBLC6-2SC6

Commit message: Updates
Parts:
- BOOT0: renamed from SW2; footprint random-keyboard-parts:PushButton_6x6mm_TH -> random-keyboard-parts:SKQG-1155865
- RESET: renamed from SW1; footprint random-keyboard-parts:PushButton_6x6mm_TH -> random-keyboard-parts:SKQG-1155865
- moved D_49 1.00 mm to (375.4, 130.7)
- moved R1 0.85 mm to (94.5, 147.6)
- turned RESET to 180 degrees
Connections:
- K_ANSIEnter1 pad 1: col13 -> col14
- K_ANSIEnter1 pad 2: Net-(D_66-Pad2) -> Net-(D_90-Pad2)
- K_ANSIShift1 pad 1: col1 -> col0
- K_ANSIShift1 pad 2: Net-(D_70-Pad2) -> Net-(D_101-Pad2)
Routing:
- net GND: track 398.3 -> 589.6 mm, vias 6 -> 13
- net col1: track 283.9 -> 264.8 mm
- net Net-(D_90-Pad2): track 10.00 -> 28.3 mm
- net Net-(D_70-Pad2): track 22.4 -> 7.61 mm
- net col0: track 291.9 -> 304.3 mm
- net Net-(D_101-Pad2): track 12.2 -> 21.7 mm
- net col14: track 194.0 -> 202.1 mm
- net col13: track 198.0 -> 191.0 mm
- net NRST: track 234.8 -> 238.6 mm, vias 2 -> 4
- net +3V3: track 309.4 -> 313.1 mm
- net row3: track 383.1 -> 386.7 mm
- net BOOT0: track 255.0 -> 257.5 mm
- net col6: track 188.9 -> 186.8 mm
- net Net-(D_49-Pad2): track 14.1 -> 15.7 mm
- net col9: track 111.4 -> 112.9 mm
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Other:
- outline, holes or cut-outs redrawn
- board text added: "6.25"
- board text added: "ANSI"
- board text added: "ISO"
- board text added: "Split"
- board text added: "Stepped"
