File: PCB/PCBV3/PCBV3.sch (KiCad schematic (older format))
At the start: 232 parts, among them SW1 SW_PUSH, SW2 SW_PUSH, U1 STM32F072CBUx, U2 MCP1700-3302E_SOT23, U3 USBLC6-2SC6

Commit message: Updates
Parts:
- SW1, SW2: footprint random-keyboard-parts:PushButton_6x6mm_TH -> random-keyboard-parts:SKQG-1155865
Connections:
- net col0: now also K_ANSIShift1.1 (COL)
- net col1: no longer K_ANSIShift1.1 (COL)
- net col13: no longer K_ANSIEnter1.1 (COL)
- net col14: now also K_ANSIEnter1.1 (COL)
- net at D_66.2 (A), K_ISO1u1R1.2 (ROW): no longer K_ANSIEnter1.2 (ROW)
- net at D_90.2 (A), K_ISOEnter1.2 (ROW): now also K_ANSIEnter1.2 (ROW)
- net at D_101.2 (A), K_ISOShift1.2 (ROW): now also K_ANSIShift1.2 (ROW)
- net at D_70.2 (A), K_ISO1uL1.2 (ROW): no longer K_ANSIShift1.2 (ROW)
Other:
- moved on the sheet: K_ANSIEnter1, K_ANSIShift1, K_ISO1u1R1, K_ISO1uL1
Changed lines of the file:
@@
 L MX_Alps_Hybrid:MX-NoLED K_ANSIShift1
 U 1 1 00000701
-P 4100 12800
-F 0 "K_ANSIShift1" H 4100 13033 60  0000 C CNN
-F 1 "KEYSW" H 4100 12700 60  0001 C CNN
-F 2 "MX_Only:MXOnly-2.25U-NoLED" H 4100 12800 60  0001 C CNN
-F 3 "" H 4100 12800 60  0000 C CNN
-	1    4100 12800
+P 3150 12750
+F 0 "K_ANSIShift1" H 3150 12983 60  0000 C CNN
+F 1 "KEYSW" H 3150 12650 60  0001 C CNN
+F 2 "MX_Only:MXOnly-2.25U-NoLED" H 3150 12750 60  0001 C CNN
+F 3 "" H 3150 12750 60  0000 C CNN
+	1    3150 12750
 	1    0    0    -1
 $EndComp
@@
 	6500 12750 6500 11750
 Wire Wire Line
-	7500 13750 7500 12750
-Wire Wire Line
 	8500 12750 8500 11750
 Wire Wire Line
@@
 Wire Wire Line
 	10500 12750 10500 11750
-Wire Wire Line
-	11500 13750 11500 12750
 Wire Wire Line
 	12500 12750 12500 11750
@@
 F 0 "SW1" H 6600 2855 50  0000 C CNN
 F 1 "SW_PUSH" H 6600 2764 50  0000 C CNN
-F 2 "random-keyboard-parts:PushButton_6x6mm_TH" H 6600 2600 60  0001 C CNN
+F 2 "random-keyboard-parts:SKQG-1155865" H 6600 2600 60  0001 C CNN
 F 3 "" H 6600 2600 60  0000 C CNN
 	1    6600 2600
@@
 F 0 "SW2" H 6600 3505 50  0000 C CNN
 F 1 "SW_PUSH" H 6600 3414 50  0000 C CNN
-F 2 "random-keyboard-parts:PushButton_6x6mm_TH" H 6600 3250 60  0001 C CNN
+F 2 "random-keyboard-parts:SKQG-1155865" H 6600 3250 60  0001 C CNN
 F 3 "" H 6600 3250 60  0000 C CNN
 	1    6600 3250
@@
 L MX_Alps_Hybrid:MX-NoLED K_ANSIEnter1
 U 1 1 00000661
-P 16100 11800
-F 0 "K_ANSIEnter1" H 16100 12033 60  0000 C CNN
-F 1 "KEYSW" H 16100 11700 60  0001 C CNN
-F 2 "MX_Only:MXOnly-2.25U-NoLED" H 16100 11800 60  0001 C CNN
-F 3 "" H 16100 11800 60  0000 C CNN
-	1    16100 11800
-	1    0    0    -1
-$EndComp
-Wire Wire Line
-	15700 12000 16050 12000
-Connection ~ 16050 12000
+P 17150 11750
+F 0 "K_ANSIEnter1" H 17150 11983 60  0000 C CNN
+F 1 "KEYSW" H 17150 11650 60  0001 C CNN
+F 2 "MX_Only:MXOnly-2.25U-NoLED" H 17150 11750 60  0001 C CNN
+F 3 "" H 17150 11750 60  0000 C CNN
+	1    17150 11750
+	1    0    0    -1
+$EndComp
 $Comp
 L Device:D_Small D_90
@@
 $EndComp
 Wire Wire Line
-	4500 9750 4500 12600
-Wire Wire Line
 	3300 12700 3500 12700
 Connection ~ 3500 12700
@@
 L MX_Alps_Hybrid:MX-NoLED K_ISO1uL1
 U 1 1 6000220A
-P 3750 12650
-F 0 "K_ISO1uL1" H 3750 12883 60  0000 C CNN
-F 1 "KEYSW" H 3750 12550 60  0001 C CNN
-F 2 "MX_Only:MXOnly-1U-NoLED" H 3750 12650 60  0001 C CNN
-F 3 "" H 3750 12650 60  0000 C CNN
-	1    3750 12650
-	1    0    0    -1
-$EndComp
-Wire Wire Line
-	3900 12600 4500 12600
-Connection ~ 4500 12600
-Wire Wire Line
-	4500 12600 4500 12750
-Wire Wire Line
-	3700 13000 4050 13000
-Connection ~ 4050 13000
-Wire Wire Line
-	16500 10750 16500 11600
+P 4100 12800
+F 0 "K_ISO1uL1" H 4100 13033 60  0000 C CNN
+F 1 "KEYSW" H 4100 12700 60  0001 C CNN
+F 2 "MX_Only:MXOnly-1U-NoLED" H 4100 12800 60  0001 C CNN
+F 3 "" H 4100 12800 60  0000 C CNN
+	1    4100 12800
+	1    0    0    -1
+$EndComp
 $Comp
 L MX_Alps_Hybrid:MX-NoLED K_ISO1u1R1
 U 1 1 5FD50D9F
-P 15750 11650
-F 0 "K_ISO1u1R1" H 15750 11883 60  0000 C CNN
-F 1 "KEYSW" H 15750 11550 60  0001 C CNN
-F 2 "MX_Only:MXOnly-1U-NoLED" H 15750 11650 60  0001 C CNN
-F 3 "" H 15750 11650 60  0000 C CNN
-	1    15750 11650
-	1    0    0    -1
-$EndComp
-Wire Wire Line
-	15900 11600 16500 11600
-Connection ~ 16500 11600
-Wire Wire Line
-	16500 11600 16500 11750
-Wire Wire Line
-	15700 11800 15700 12000
-Wire Wire Line
-	3700 12800 3700 13000
+P 16100 11800
+F 0 "K_ISO1u1R1" H 16100 12033 60  0000 C CNN
+F 1 "KEYSW" H 16100 11700 60  0001 C CNN
+F 2 "MX_Only:MXOnly-1U-NoLED" H 16100 11800 60  0001 C CNN
+F 3 "" H 16100 11800 60  0000 C CNN
+	1    16100 11800
+	1    0    0    -1
+$EndComp
 Text GLabel 9950 4250 2    50   Input ~ 0
 D-
+Wire Wire Line
+	7500 13750 7500 12750
+Wire Wire Line
+	11500 13750 11500 12750
+Connection ~ 3300 12700
+Connection ~ 3100 12900
+Wire Wire Line
+	4500 9750 4500 12750
+Connection ~ 17300 11700
+Connection ~ 17100 11900
+Wire Wire Line
+	16500 10750 16500 11750
 $EndSCHEMATC
