File: Plate/PlateV1/Plate/Plate.sch (KiCad schematic (older format))
At the start: 2 parts

Commit message: Updates
Parts:
- removed R1, R2: R_Small, Resistor_SMD:R_0603_1608Metric, symbol Device:R_Small
- added G1: Graphic, Keybage_MX_Cutout:MX_Cutout_1u, symbol keybage:Graphic
Changed lines of the file:
@@
 $EndDescr
 $Comp
-L Device:R_Small R1
-U 1 1 5FA59ED1
-P 3600 2850
-F 0 "R1" H 3659 2896 50  0000 L CNN
-F 1 "R_Small" H 3659 2805 50  0000 L CNN
-F 2 "Resistor_SMD:R_0603_1608Metric" H 3600 2850 50  0001 C CNN
-F 3 "~" H 3600 2850 50  0001 C CNN
-	1    3600 2850
+L keybage:Graphic G1
+U 1 1 5FC1FBF6
+P 5650 4000
+F 0 "G1" H 5728 4046 50  0000 L CNN
+F 1 "Graphic" H 5728 3955 50  0000 L CNN
+F 2 "Keybage_MX_Cutout:MX_Cutout_1u" H 5700 4000 50  0001 C CNN
+F 3 "" H 5700 4000 50  0001 C CNN
+	1    5650 4000
 	1    0    0    -1
 $EndComp
-$Comp
-L Device:R_Small R2
-U 1 1 5FA6E719
-P 4350 2800
-F 0 "R2" H 4409 2846 50  0000 L CNN
-F 1 "R_Small" H 4409 2755 50  0000 L CNN
-F 2 "Resistor_SMD:R_0603_1608Metric" H 4350 2800 50  0001 C CNN
-F 3 "~" H 4350 2800 50  0001 C CNN
-	1    4350 2800
-	1    0    0    -1
-$EndComp
